File: PCB/Overdrive/Overdrive.kicad_pcb (KiCad board)
At the start: 2 copper layers, 3 parts

Commit message: A
Parts:
- added C10: C, Capacitor_THT:CP_Radial_Tantal_D5.5mm_P5.00mm, F.Cu at (140.5, 57.5)
- added C11: C, Capacitor_THT:CP_Radial_Tantal_D5.5mm_P5.00mm, F.Cu at (213.0, 98.5)
- added C12: C, Capacitor_THT:CP_Radial_Tantal_D5.5mm_P5.00mm, F.Cu at (156.2, 57.5)
- added C13: C, Capacitor_THT:CP_Radial_Tantal_D5.5mm_P5.00mm, F.Cu at (164.0, 57.5)
- added C2: C, Capacitor_THT:CP_Radial_Tantal_D5.5mm_P5.00mm, F.Cu at (92.5, 141.0)
- added C4: C, Capacitor_THT:CP_Radial_Tantal_D5.5mm_P5.00mm, F.Cu at (52.0, 169.5)
- added C_ADC1: ~, Capacitor_THT:CP_Radial_D10.0mm_P5.00mm, F.Cu at (56.1, 182.5)
- added C_TL072_1: C, Capacitor_THT:CP_Radial_Tantal_D5.5mm_P5.00mm, F.Cu at (171.9, 18.6)
- added C_TL072_2: C, Capacitor_THT:CP_Radial_Tantal_D5.5mm_P5.00mm, F.Cu at (55.5, 147.0)
- added C_entrada1: C, Capacitor_THT:CP_Radial_Tantal_D5.5mm_P5.00mm, F.Cu at (47.5, 108.0)
- added C_salida1: ~, Capacitor_THT:CP_Radial_D10.0mm_P5.00mm, F.Cu at (180.6, 32.0)
- added C_sbt1: C, Capacitor_THT:CP_Radial_Tantal_D5.5mm_P5.00mm, F.Cu at (132.7, 57.5)
- added C_sovdr1: C, Capacitor_THT:CP_Radial_Tantal_D5.5mm_P5.00mm, F.Cu at (117.0, 57.5)
- added C_spwm1: C, Capacitor_THT:CP_Radial_Tantal_D5.5mm_P5.00mm, F.Cu at (124.8, 57.5)
- added C_vref1: ~, Capacitor_THT:CP_Radial_D10.0mm_P5.00mm, F.Cu at (88.6, 117.0)
- added J1: Alimentación, TerminalBlock:TerminalBlock_MaiXu_MX126-5.0-02P_1x02_P5.00mm, F.Cu at (88.0, 100.0)
- added J2: Entrada, TerminalBlock:TerminalBlock_MaiXu_MX126-5.0-02P_1x02_P5.00mm, F.Cu at (36.0, 111.5)
- added J3: Salida, TerminalBlock:TerminalBlock_MaiXu_MX126-5.0-02P_1x02_P5.00mm, F.Cu at (210.3, 25.8)
- added J4: LM1117_3.3V, TerminalBlock:TerminalBlock_MaiXu_MX126-5.0-03P_1x03_P5.00mm, F.Cu at (67.0, 100.0)
- added J6: BT, TerminalBlock:TerminalBlock_MaiXu_MX126-5.0-04P_1x04_P5.00mm, F.Cu at (292.6, 106.6)
- added R1: R_US, Resistor_THT:R_Axial_DIN0207_L6.3mm_D2.5mm_P10.16mm_Horizontal, F.Cu at (55.4, 164.0)
- added R10: 4.7k, Resistor_THT:R_Axial_DIN0207_L6.3mm_D2.5mm_P10.16mm_Horizontal, F.Cu at (46.5, 177.6)
- added R11: 100k, Resistor_THT:R_Axial_DIN0207_L6.3mm_D2.5mm_P10.16mm_Horizontal, F.Cu at (265.2, 68.4)
- added R12: R_US, Resistor_THT:R_Axial_DIN0207_L6.3mm_D2.5mm_P10.16mm_Horizontal, F.Cu at (83.1, 111.0)
- added R13: R_US, Resistor_THT:R_Axial_DIN0207_L6.3mm_D2.5mm_P10.16mm_Horizontal, F.Cu at (246.6, 55.1)
- added R14: R_US, Resistor_THT:R_Axial_DIN0207_L6.3mm_D2.5mm_P10.16mm_Horizontal, F.Cu at (247.1, 68.3)
- added R15: R_US, Resistor_THT:R_Axial_DIN0207_L6.3mm_D2.5mm_P10.16mm_Horizontal, F.Cu at (248.1, 75.3)
- added R16: R_US, Resistor_THT:R_Axial_DIN0207_L6.3mm_D2.5mm_P10.16mm_Horizontal, F.Cu at (82.6, 123.5)
- added R2: R_US, Resistor_THT:R_Axial_DIN0207_L6.3mm_D2.5mm_P10.16mm_Horizontal, F.Cu at (72.4, 117.5)
- added R3: R_US, Resistor_THT:R_Axial_DIN0207_L6.3mm_D2.5mm_P10.16mm_Horizontal, F.Cu at (194.7, 63.4)
- added R4: R_US, Resistor_THT:R_Axial_DIN0207_L6.3mm_D2.5mm_P10.16mm_Horizontal, F.Cu at (46.4, 123.5)
- added R5: R_US, Resistor_THT:R_Axial_DIN0207_L6.3mm_D2.5mm_P10.16mm_Horizontal, F.Cu at (84.5, 146.1)
- added R6: R_US, Resistor_THT:R_Axial_DIN0207_L6.3mm_D2.5mm_P10.16mm_Horizontal, F.Cu at (79.0, 146.6)
- added R7: 100k, Resistor_THT:R_Axial_DIN0207_L6.3mm_D2.5mm_P10.16mm_Horizontal, F.Cu at (264.7, 51.9)
- added R8: R_US, Resistor_THT:R_Axial_DIN0207_L6.3mm_D2.5mm_P10.16mm_Horizontal, F.Cu at (64.9, 145.5)
- added R9: 100k, Resistor_THT:R_Axial_DIN0207_L6.3mm_D2.5mm_P10.16mm_Horizontal, F.Cu at (35.5, 159.1)
- added RV1: P_rspb, Potentiometer_THT:Potentiometer_Alps_RK163_Single_Horizontal, F.Cu at (190.1, 123.3)
- added RV2: P_ovdr, Potentiometer_THT:Potentiometer_Alps_RK163_Single_Horizontal, F.Cu at (209.6, 123.3)
- added RV3: Pote_Doble, Potentiometer_THT:Potentiometer_Alps_RK163_Dual_Horizontal, F.Cu at (74.0, 157.8)
- added RV4: P_adc, Potentiometer_THT:Potentiometer_Alps_RK163_Single_Horizontal, F.Cu at (36.0, 169.5)
- added RV5: P_bt, Potentiometer_THT:Potentiometer_Alps_RK163_Single_Horizontal, F.Cu at (254.1, 121.1)
- added R_vref_1: 10k, Resistor_THT:R_Axial_DIN0207_L6.3mm_D2.5mm_P10.16mm_Horizontal, F.Cu at (64.0, 107.9)
- added R_vref_2: 10k, Resistor_THT:R_Axial_DIN0207_L6.3mm_D2.5mm_P10.16mm_Horizontal, F.Cu at (64.0, 122.4)
- added SW1: BT_sw, Connector_PinSocket_2.54mm:PinSocket_2x03_P2.54mm_Vertical, F.Cu at (208.6, 45.1)
- added SW2: BT_sw, Connector_PinSocket_2.54mm:PinSocket_2x03_P2.54mm_Horizontal, F.Cu at (48.2, 138.9)
- added U1: TL072, Package_DIP:DIP-8_W7.62mm_Socket, F.Cu at (205.3, 59.5)
- added U2: TL072, Package_DIP:DIP-8_W7.62mm_Socket, F.Cu at (44.7, 151.7)
- moved A1 271.9 mm to (283.3, 58.1)
- moved D1 161.0 mm to (60.0, 158.5), turned to 90 degrees
- moved D2 151.1 mm to (64.0, 150.9), turned to -90 degrees
Routing:
- added copper zone on B.Cu, net GND

Commit message: A
Parts:
- J4: footprint TerminalBlock:TerminalBlock_MaiXu_MX126-5.0-03P_1x03_P5.00mm -> Connector_PinHeader_2.54mm:PinHeader_1x03_P2.54mm_Vertical
- J6: footprint TerminalBlock:TerminalBlock_MaiXu_MX126-5.0-04P_1x04_P5.00mm -> Connector_PinHeader_2.54mm:PinHeader_1x04_P2.54mm_Vertical
- RV1, RV2, RV4, RV5: footprint Potentiometer_THT:Potentiometer_Alps_RK163_Single_Horizontal -> Connector_PinHeader_2.54mm:PinHeader_1x03_P2.54mm_Vertical
- RV3: footprint Potentiometer_THT:Potentiometer_Alps_RK163_Dual_Horizontal -> Connector_PinSocket_2.54mm:PinSocket_2x03_P2.54mm_Vertical
- SW2: footprint Connector_PinSocket_2.54mm:PinSocket_2x03_P2.54mm_Horizontal -> Connector_PinSocket_2.54mm:PinSocket_2x03_P2.54mm_Vertical
- moved A1 234.0 mm to (60.0, 128.1), turned to 90 degrees
- moved R13 190.1 mm to (106.9, 184.0), turned to 180 degrees
- moved R11 182.0 mm to (94.1, 130.6), turned to 0 degrees
- moved J6 181.1 mm to (122.2, 167.8), turned to 180 degrees
- moved R7 177.4 mm to (104.0, 127.2), turned to 0 degrees
- moved J3 174.3 mm to (119.2, 174.4), turned to -90 degrees
- moved R14 172.0 mm to (98.1, 154.4)
- moved R15 168.8 mm to (96.6, 149.8), turned to 90 degrees
- moved C_salida1 162.5 mm to (105.0, 175.8)
- moved C_TL072_1 161.4 mm to (93.3, 159.6), turned to 180 degrees
- moved R3 157.9 mm to (84.0, 176.1)
- moved U1 157.6 mm to (91.2, 168.2)
- moved SW1 155.3 mm to (105.1, 160.7)
- moved RV5 147.1 mm to (109.0, 145.2), turned to 180 degrees
- moved RV2 146.1 mm to (78.0, 186.8)
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Connections:
- A1 pad 13: Net-(A1-GND-Pad13) -> GND
- A1 pad 18: Net-(A1-GND-Pad13) -> GND
- A1 pad 23: Net-(A1-GND-Pad13) -> GND
- A1 pad 28: Net-(A1-GND-Pad13) -> GND
- A1 pad 3: Net-(A1-GND-Pad13) -> GND
- A1 pad 38: Net-(A1-GND-Pad13) -> GND
- A1 pad 8: Net-(A1-GND-Pad13) -> GND
Routing:
- net Vref: track 0.00 -> 190.4 mm
- net Vcc: track 0.00 -> 121.7 mm
- net Net-(D1-A): track 0.00 -> 80.0 mm
- net Net-(U1A--): track 0.00 -> 78.7 mm
- net ADC_IN: track 0.00 -> 66.8 mm
- net Net-(SW2A-A): track 0.00 -> 37.9 mm
- net Net-(U1A-+): track 0.00 -> 31.7 mm
- net Net-(U2A--): track 0.00 -> 31.1 mm
- net Net-(SW2A-B): track 0.00 -> 28.3 mm
- net Net-(D1-K): track 0.00 -> 24.7 mm
- net Net-(SW1A-A): track 0.00 -> 24.0 mm
- net Net-(C13-Pad2): track 0.00 -> 22.6 mm
- net Net-(U1B-+): track 0.00 -> 20.7 mm
- net PWM_out: track 0.00 -> 20.6 mm
- net Net-(J6-Pin_4): track 0.00 -> 18.5 mm
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Other:
- board outline added: 114 x 85.4 mm
