File: PCB/Overdrive/Overdrive.kicad_sch (KiCad schematic)
At the start: 25 parts, among them J1 Alimentación, J2 Entrada, J3 Salida, SW1 SW_DPDT_x2, U1 TL072, U2 TL072

Commit message: A
Parts:
- removed C3: C_US, symbol Device:C_US
- added A1: RaspberryPi_Pico, Module:RaspberryPi_Pico_Common_Unspecified, symbol MCU_Module:RaspberryPi_Pico
- added C10, C11, C12, C13, C2, C8, C9: C, Capacitor_THT:CP_Axial_L11.0mm_D6.0mm_P18.00mm_Horizontal, symbol Device:C
- added C_ADC1: ~, Capacitor_THT:CP_Radial_D25.0mm_P10.00mm_3pin_SnapIn, symbol Device:C_US
- added J4: LM1117_3.3V, symbol Connector:Conn_01x03_Pin
- added J6: BT, symbol Connector:Conn_01x04_Socket
- added R10: 4.7k, symbol Device:R_US
- added R11, R9: 100k, symbol Device:R_US
- added R12, R13, R14, R15, R16, R2, R3: R_US, symbol Device:R_US
- added RV4, RV5: P_tono, symbol Device:R_Potentiometer_US
- C1, C4, C5: footprint (none) -> Capacitor_THT:CP_Axial_L11.0mm_D6.0mm_P18.00mm_Horizontal
- C_salida1: renamed from C6; value C_US -> ~; footprint (none) -> Capacitor_THT:CP_Radial_D25.0mm_P10.00mm_3pin_SnapIn
- C_vref1: renamed from C2; value C_US -> ~; footprint (none) -> Capacitor_THT:CP_Radial_D25.0mm_P10.00mm_3pin_SnapIn
- R7: value R_US -> 100k
- R_vref_1: renamed from R3; value R_US -> 10k
- R_vref_2: renamed from R2; value R_US -> 10k
- SW1: value SW_DPDT_x2 -> BT_sw
Connections:
- net GND: now also SW1.3 (C), SW1.6 (C), C10.1, C11.1, C2.1, C_ADC1.2, J4.2 (Pin_2), J6.2 (Pin_2), J6.3 (Pin_3), R13.1, R14.1, R15.1; no longer C5.1
- net Vref: now also R12.2, R16.2, R2.2; no longer U1.3 (+)
- net at R8.1, RV3.4: now also D1.2 (A), D2.1 (K), RV2.1, RV3.2, RV3.3, U2.7; no longer RV1.1
- net at C5.2: now also RV2.3; no longer RV1.2
- net at U1.1, U1.5 (+): now also R3.2; no longer RV2.1, RV2.2
- net at R6.1, R8.2, RV3.5: no longer SW1.4 (A)
- net at R5.2, R6.2: now also C2.2
- net at U2.5 (+): now also C1.2, R4.1, U2.3 (+); no longer SW1.1 (A)
- net at R7.1: now also C11.2, R11.2; no longer SW1.5 (B)
- net 9V renamed Vcc
- net Vcc: now also SW1.4 (A), J4.3 (Pin_3); no longer R_vref_1.1
- new net: C8.1, R14.2
- new net: C8.2, RV1.3
- new net: C12.1, R7.2
- new net: J6.1 (Pin_1), SW1.5 (B)
- new net: J6.4 (Pin_4), SW1.2 (B)
- new net: C12.2, R12.1, RV1.1
- new net: C5.1, R13.2
- new net: C13.2, R16.1, RV5.1
- new net: C9.1, R15.2
- new net: RV1.2, RV5.2
- new net: C9.2, RV5.3
- new net: C13.1, SW1.1 (A)
- new net: R3.1, RV2.2, U1.2 (-)
- new net: R2.1, U1.3 (+)
- new net: R9.1, RV4.2, RV4.3, U2.2 (-)
- new net: A1.13 (GND), A1.18 (GND), A1.23 (GND), A1.28 (GND), A1.3 (GND), A1.38 (GND), A1.8 (GND)
- new net: C_ADC1.1, R10.1
- new net: R10.2, RV4.1
- new net 3.3V: J4.1 (Pin_1), R_vref_1.1
- new net ADC_IN: A1.31 (GPIO26_ADC0), R9.2, U2.1
- new net PWM_out: A1.19 (GPIO14), C10.2, R11.1
Other:
- moved on the sheet: C1, C4, C_salida1, D1, D2, J2, J3, R1, R4, R5, R6, R8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

Commit message: A
Parts:
- C_ADC1, C_salida1, C_vref1: value ~ -> (none)
- R1, R10, R11, R12, R13, R14, R15, R16, R2, R3, R4, R5, R6, R7, R8, R9, R_vref_1, R_vref_2: footprint (none) -> Resistor_THT:R_Axial_DIN0207_L6.3mm_D2.5mm_P10.16mm_Horizontal

Commit message: A
Parts:
- added C_TL072_1, C_TL072_2: C, Capacitor_THT:CP_Radial_Tantal_D5.5mm_P5.00mm, symbol Device:C
- added SW2: BT_sw, Connector_PinSocket_2.54mm:PinSocket_2x03_P2.54mm_Horizontal, symbol Switch:SW_DPDT_x2
- C10, C11, C12, C13, C2, C4: footprint Capacitor_THT:CP_Axial_L11.0mm_D6.0mm_P18.00mm_Horizontal -> Capacitor_THT:CP_Radial_Tantal_D5.5mm_P5.00mm
- C_ADC1, C_salida1, C_vref1: footprint Capacitor_THT:CP_Radial_D25.0mm_P10.00mm_3pin_SnapIn -> Capacitor_THT:CP_Radial_D10.0mm_P5.00mm
- C_entrada1: renamed from C1; footprint Capacitor_THT:CP_Axial_L11.0mm_D6.0mm_P18.00mm_Horizontal -> Capacitor_THT:CP_Radial_Tantal_D5.5mm_P5.00mm
- C_sbt1: renamed from C9; footprint Capacitor_THT:CP_Axial_L11.0mm_D6.0mm_P18.00mm_Horizontal -> Capacitor_THT:CP_Radial_Tantal_D5.5mm_P5.00mm
- C_sovdr1: renamed from C5; footprint Capacitor_THT:CP_Axial_L11.0mm_D6.0mm_P18.00mm_Horizontal -> Capacitor_THT:CP_Radial_Tantal_D5.5mm_P5.00mm
- C_spwm1: renamed from C8; footprint Capacitor_THT:CP_Axial_L11.0mm_D6.0mm_P18.00mm_Horizontal -> Capacitor_THT:CP_Radial_Tantal_D5.5mm_P5.00mm
- J1, J2, J3: footprint (none) -> TerminalBlock:TerminalBlock_MaiXu_MX126-5.0-02P_1x02_P5.00mm
- J4: footprint (none) -> TerminalBlock:TerminalBlock_MaiXu_MX126-5.0-03P_1x03_P5.00mm
- J6: footprint (none) -> TerminalBlock:TerminalBlock_MaiXu_MX126-5.0-04P_1x04_P5.00mm
- RV1: value P_tono -> P_rspb; footprint (none) -> Potentiometer_THT:Potentiometer_Alps_RK163_Single_Horizontal
- RV2: value P_tono -> P_ovdr; footprint (none) -> Potentiometer_THT:Potentiometer_Alps_RK163_Single_Horizontal
- RV3: footprint (none) -> Potentiometer_THT:Potentiometer_Alps_RK163_Dual_Horizontal
- RV4: value P_tono -> P_adc; footprint (none) -> Potentiometer_THT:Potentiometer_Alps_RK163_Single_Horizontal
- RV5: value P_tono -> P_bt; footprint (none) -> Potentiometer_THT:Potentiometer_Alps_RK163_Single_Horizontal
- SW1: footprint (none) -> Connector_PinSocket_2.54mm:PinSocket_2x03_P2.54mm_Vertical
- U1, U2: footprint (none) -> Package_DIP:DIP-8_W7.62mm_Socket
Connections:
- net GND: now also C_TL072_1.1, C_TL072_2.1
- net Vcc: now also C_TL072_1.2, C_TL072_2.2
- net at C_entrada1.2, R4.1, U2.5 (+): now also SW2.1 (A); no longer U2.3 (+)
- net at D1.2 (A), D2.1 (K), R8.1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: now also SW2.3 (C)
- new net: SW2.2 (B), U2.3 (+)
Other:
- moved on the sheet: C_entrada1, J2, R4, U2A

Commit message: A
Parts:
- J4: footprint TerminalBlock:TerminalBlock_MaiXu_MX126-5.0-03P_1x03_P5.00mm -> Connector_PinHeader_2.54mm:PinHeader_1x03_P2.54mm_Vertical
- J6: footprint TerminalBlock:TerminalBlock_MaiXu_MX126-5.0-04P_1x04_P5.00mm -> Connector_PinHeader_2.54mm:PinHeader_1x04_P2.54mm_Vertical
- RV1, RV2, RV4, RV5: footprint Potentiometer_THT:Potentiometer_Alps_RK163_Single_Horizontal -> Connector_PinHeader_2.54mm:PinHeader_1x03_P2.54mm_Vertical
- RV3: footprint Potentiometer_THT:Potentiometer_Alps_RK163_Dual_Horizontal -> Connector_PinSocket_2.54mm:PinSocket_2x03_P2.54mm_Vertical
- SW2: footprint Connector_PinSocket_2.54mm:PinSocket_2x03_P2.54mm_Horizontal -> Connector_PinSocket_2.54mm:PinSocket_2x03_P2.54mm_Vertical
Connections:
- net GND: now also A1.13 (GND), A1.18 (GND), A1.23 (GND), A1.28 (GND), A1.3 (GND), A1.38 (GND), A1.8 (GND)
Changed lines of the file:
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@@
 			)
 		)
-		(property "Footprint" "TerminalBlock:TerminalBlock_MaiXu_MX126-5.0-03P_1x03_P5.00mm"
+		(property "Footprint" "Connector_PinHeader_2.54mm:PinHeader_1x03_P2.54mm_Vertical"
 			(at 60.96 156.21 0)
 			(hide yes)
@@
 			)
 		)
-		(property "Footprint" "TerminalBlock:TerminalBlock_MaiXu_MX126-5.0-04P_1x04_P5.00mm"
+		(property "Footprint" "Connector_PinHeader_2.54mm:PinHeader_1x04_P2.54mm_Vertical"
 			(at 17.78 146.05 0)
 			(hide yes)
@@
 			)
 		)
-		(property "Footprint" "Potentiometer_THT:Potentiometer_Alps_RK163_Single_Horizontal"
+		(property "Footprint" "Connector_PinHeader_2.54mm:PinHeader_1x03_P2.54mm_Vertical"
 			(at 113.03 66.04 0)
 			(hide yes)
@@
 			)
 		)
-		(property "Footprint" "Potentiometer_THT:Potentiometer_Alps_RK163_Single_Horizontal"
+		(property "Footprint" "Connector_PinHeader_2.54mm:PinHeader_1x03_P2.54mm_Vertical"
 			(at 113.03 123.19 0)
 			(hide yes)
@@
 			)
 		)
-		(property "Footprint" "Connector_PinSocket_2.54mm:PinSocket_2x03_P2.54mm_Horizontal"
+		(property "Footprint" "Connector_PinSocket_2.54mm:PinSocket_2x03_P2.54mm_Vertical"
 			(at 38.1 72.39 0)
 			(hide yes)
@@
 			(at 38.1 72.39 0)
 			(hide yes)
-			(show_name no)
+			(show_name yes)
 			(do_not_autoplace no)
 			(effects
@@
 			)
 		)
-		(property "Footprint" "Connector_PinSocket_2.54mm:PinSocket_2x03_P2.54mm_Horizontal"
+		(property "Footprint" "Connector_PinSocket_2.54mm:PinSocket_2x03_P2.54mm_Vertical"
 			(at 134.62 20.32 0)
 			(hide yes)
@@
 			)
 		)
-		(property "Footprint" "Potentiometer_THT:Potentiometer_Alps_RK163_Dual_Horizontal"
+		(property "Footprint" "Connector_PinSocket_2.54mm:PinSocket_2x03_P2.54mm_Vertical"
 			(at 50.8 121.92 0)
 			(hide yes)
@@
 			)
 		)
-		(property "Footprint" "Potentiometer_THT:Potentiometer_Alps_RK163_Dual_Horizontal"
+		(property "Footprint" "Connector_PinSocket_2.54mm:PinSocket_2x03_P2.54mm_Vertical"
 			(at 68.58 96.52 0)
 			(hide yes)
@@
 			)
 		)
-		(property "Footprint" "Potentiometer_THT:Potentiometer_Alps_RK163_Single_Horizontal"
+		(property "Footprint" "Connector_PinHeader_2.54mm:PinHeader_1x03_P2.54mm_Vertical"
 			(at 113.03 95.25 0)
 			(hide yes)
@@
 	(symbol
 		(lib_id "power:GND")
+		(at 248.92 87.63 0)
+		(mirror y)
+		(unit 1)
+		(body_style 1)
+		(exclude_from_sim no)
+		(in_bom yes)
+		(on_board yes)
+		(in_pos_files yes)
+		(dnp no)
+		(fields_autoplaced yes)
+		(property "Reference" "#PWR022"
+			(at 248.92 93.98 0)
+			(hide yes)
+			(show_name no)
+			(do_not_autoplace no)
+			(effects
+				(font
+					(size 1.27 1.27)
+				)
+			)
+		)
+		(property "Value" "GND"
+			(at 248.92 92.71 0)
+			(show_name no)
+			(do_not_autoplace no)
+			(effects
+				(font
+					(size 1.27 1.27)
+				)
+			)
+		)
+		(property "Footprint" ""
+			(at 248.92 87.63 0)
+			(hide yes)
+			(show_name no)
+			(do_not_autoplace no)
+			(effects
+				(font
+					(size 1.27 1.27)
+				)
+			)
+		)
+		(property "Datasheet" ""
+			(at 248.92 87.63 0)
+			(hide yes)
+			(show_name no)
+			(do_not_autoplace no)
+			(effects
+				(font
+					(size 1.27 1.27)
+				)
+			)
+		)
+		(property "Description" "Power symbol creates a global label with name \"GND\" , ground"
+			(at 248.92 87.63 0)
+			(hide yes)
+			(show_name no)
+			(do_not_autoplace no)
+			(effects
+				(font
+					(size 1.27 1.27)
+				)
+			)
+		)
+		(pin "1"
+		)
+		(instances
+			(project "Overdrive"
+				(path "/6ab4e771-ed81-43fb-b5c5-ca1b3b0e4bae"
+					(reference "#PWR022")
+					(unit 1)
+				)
+			)
+		)
+	)
+	(symbol
+		(lib_id "power:GND")
 		(at 25.4 146.05 90)
 		(unit 1)
@@
 			)
 		)
-		(property "Footprint" "Potentiometer_THT:Potentiometer_Alps_RK163_Single_Horizontal"
+		(property "Footprint" "Connector_PinHeader_2.54mm:PinHeader_1x03_P2.54mm_Vertical"
 			(at 34.29 55.88 0)
 			(hide yes)

Commit message: A
Parts:
- removed C13, C_sbt1: C, Capacitor_THT:CP_Radial_Tantal_D5.5mm_P5.00mm, symbol Device:C
- removed J6: BT, Connector_PinHeader_2.54mm:PinHeader_1x04_P2.54mm_Vertical, symbol Connector:Conn_01x04_Socket
- removed RV5: P_bt, Connector_PinHeader_2.54mm:PinHeader_1x03_P2.54mm_Vertical, symbol Device:R_Potentiometer_US
- removed SW1: BT_sw, Connector_PinSocket_2.54mm:PinSocket_2x03_P2.54mm_Vertical, symbol Switch:SW_DPDT_x2
- added D3, D4: LED, LED_THT:LED_D5.0mm_FlatTop, symbol Device:LED
- added SW3: RotaryEncoder_Switch, symbol Device:RotaryEncoder_Switch
Connections:
- net 3.3V: now also J4.2 (Pin_2); no longer J4.1 (Pin_1)
- net GND: now also J4.1 (Pin_1), R15.2, R16.2; no longer J4.2 (Pin_2), R15.1
- net Vcc: now also A1.39 (VSYS), SW2.5 (B)
- net Vref: no longer R16.2
- net at R16.1: now also D4.1 (K)
- net at RV1.2: now also R3.1, RV2.2, U1.2 (-)
- net at SW2.4 (A): now also D4.2 (A)
- net at SW2.6 (C): now also D3.2 (A)
- new net: D3.1 (K), R15.1
Other:
- moved on the sheet: A1, SW2B
