File: PCB/Overdrive/Overdrive.kicad_sch (KiCad schematic)
At the start: 54 parts, among them J1 Alimentación, J2 Entrada, J3 Salida, J4 LM1117_3.3V, SW2 BT_sw, SW3 RotaryEncoder_Switch, U1 TL072, U2 TL072

Commit message: A
Parts:
- added D8: LED, LED_THT:LED_D5.0mm_FlatTop, symbol Device:LED
- added FS5, J7: OUT, Connector_PinHeader_2.54mm:PinHeader_1x01_P2.54mm_Vertical, symbol Connector:Conn_01x01_Pin
- added J10: FS2, Connector_PinHeader_2.54mm:PinHeader_1x01_P2.54mm_Vertical, symbol Connector:Conn_01x01_Pin
- added J11: FS3, Connector_PinHeader_2.54mm:PinHeader_1x01_P2.54mm_Vertical, symbol Connector:Conn_01x01_Pin
- added J12: FS6, Connector_PinHeader_2.54mm:PinHeader_1x01_P2.54mm_Vertical, symbol Connector:Conn_01x01_Pin
- added J13: FS4, Connector_PinHeader_2.54mm:PinHeader_1x01_P2.54mm_Vertical, symbol Connector:Conn_01x01_Pin
- added J5: OVD, Connector_PinHeader_2.54mm:PinHeader_1x01_P2.54mm_Vertical, symbol Connector:Conn_01x01_Pin
- added J6: PWM, Connector_PinHeader_2.54mm:PinHeader_1x01_P2.54mm_Vertical, symbol Connector:Conn_01x01_Pin
- added J8: ADC_in, Connector_PinHeader_2.54mm:PinHeader_1x01_P2.54mm_Vertical, symbol Connector:Conn_01x01_Pin
- added J9: FS1, Connector_PinHeader_2.54mm:PinHeader_1x01_P2.54mm_Vertical, symbol Connector:Conn_01x01_Pin
- added R20: R_US, Resistor_THT:R_Axial_DIN0207_L6.3mm_D2.5mm_P10.16mm_Horizontal, symbol Device:R_US
Connections:
- net ADC_IN: now also J8.1 (Pin_1)
- net GND: now also D8.2 (A), J11.1 (Pin_1)
- net PWM_out: now also J6.1 (Pin_1)
- net Vcc: now also J10.1 (Pin_1)
- net at R6.1, R8.2, RV3.5: now also RV2.1, J5.1 (Pin_1)
- net at D1.2 (A), D2.1 (K), R8.1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: no longer RV2.1
- net In: now reaches C_entrada1.1, J2.2 (Pin_2)
- net In: now also J13.1 (Pin_1)
- net at J3.1 (Pin_1): now also J12.1 (Pin_1); no longer C_salida1.2
- new net: D8.1 (K), R20.1
- new net: J9.1 (Pin_1), R20.2
- new net Out_p: C_salida1.2, FS5.1 (Pin_1), J7.1 (Pin_1)
Other:
- moved on the sheet: J3
