File: PCB/Overdrive/Overdrive_V2.kicad_sch (KiCad schematic)
At the start: 54 parts, among them J1 Alimentación, J2 Entrada, J3 Salida, J4 LM1117_3.3V, SW2 BT_sw, SW3 RotaryEncoder_Switch, U1 TL072, U2 TL072

Commit message: A
Parts:
- removed D5, D6, D7: LED, LED_THT:LED_D5.0mm_FlatTop, symbol Device:LED
- removed R17, R18, R19: R_US, Resistor_THT:R_Axial_DIN0207_L6.3mm_D2.5mm_P10.16mm_Horizontal, symbol Device:R_US
- SW3: footprint Connector_PinSocket_2.54mm:PinSocket_1x05_P2.54mm_Vertical -> Rotary_Encoder:RotaryEncoder_Alps_EC11E-Switch_Vertical_H20mm_CircularMountingHoles
Other:
- moved on the sheet: SW2B
